File: hardware/ss.brd (EAGLE design)
At the start: 70 x 56.5 mm, 76 parts, among them IC1 DS3231, Q1 BSS138, Q3 si2305cd, Q4 si2305cd, Q5 8MHz, Q6 si2305cd, U1 SPX5205 3v3, U17 AVR_SPI_PRG_6PTH, U2 CN3083, U3 SPX5205 3v3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

Commit message: latest
Parts:
- removed BAT1: 3v, SparkFun:BATTCON_12MM
- removed Q3: si2305cd, Simplex-DiscreteSemi:SOT23-3_POWER
- added C22: 100nF, rcl:C0805
- added JP11: analog, SparkFun:1X06
- added JP14: digital, SparkFun-Connectors:1X07
- added JP8: JUMPER-3SMD, SparkFun-Passives:SJ_3
- added JP9: Kterm, SparkFun:1X02
- added Q2: si2305cd, Simplex-DiscreteSemi:SOT23-3_POWER
- added R16: 100k, rcl:R0805W
- added SJ3, SJ4: (no value), SparkFun-Passives:SJ_2S-TRACE
- added T1: BC846, transistor:SOT23
- added U$3: MAX6675, SparkFun-AnalogIC:SO08-MAX6675
- JP4: value uC -> M01PTH; device SparkFun:1X02 -> SparkFun-Connectors:1X01
- JP5: value digital -> 3v Li bat; device SparkFun-Connectors:1X08 -> SparkFun:1X02
- JP6: value analog -> rxtx; device SparkFun-Connectors:1X06 -> SparkFun:1X02
- LED1: value red -> charging; device SparkFun:LED-0603 -> led:CHIP-LED0805
- LED2: value green -> full; device SparkFun:LED-0603 -> led:CHIP-LED0805
- LED4: device SparkFun:LED-0603 -> led:CHIP-LED0805
- moved R14 221.3 mm to (5.30, 21.9), turned to 270 degrees
- moved SJ1 219.6 mm to (7.80, 37.9)
- moved C21 218.9 mm to (11.2, 37.9), turned to 180 degrees
- moved R7 216.2 mm to (48.3, 30.6), turned to 180 degrees
- moved R9 215.4 mm to (3.20, 21.9), turned to 270 degrees
- moved JP5 211.0 mm to (22.0, 33.7), turned to 90 degrees
- moved Q5 208.2 mm to (53.2, 53.3), turned to 270 degrees
- moved LED4 206.6 mm to (3.70, 16.1), turned to 90 degrees
- moved R8 205.3 mm to (7.50, 16.0)
- moved R2 204.8 mm to (28.5, 46.5), turned to 90 degrees
- moved C27 204.7 mm to (51.6, 47.7), turned to 90 degrees
- moved U$7 204.2 mm to (32.2, 58.3)
- moved SJ2 202.2 mm to (10.8, 15.9)
- moved R23 202.0 mm to (32.2, 54.8)
- moved JP6 199.7 mm to (10.5, 21.7), turned to 180 degrees
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Connections:
- removed net D4: JP5.2, U5.2
- removed net N$4: IC1.15, JP4.2, R13.2
- removed net N$6: IC1.16, JP4.1, R10.2
- removed net XBEE_IN: C18.1, C20.1, Q3.3, U3.1, U3.3
- removed net XBEE_PWR_SW: Q3.1, R1.2, U$2.9, U5.25
- new net A2: JP8.2, JP8.3, U5.25
- new net A3: JP11.4, U5.26
- new net N$100: C16.1, C17.1, Q2.2, R1.2, SJ3.2, U3.5
- new net N$26: R7.1, T1.1
- new net N$27: Q4.1, R16.2, T1.3
- new net N$29: JP9.1, U$3.3
- new net N$30: JP9.2, U$3.2
- new net XBEE_HIB: SJ4.1, U$2.9
- new net XBEE_PWR_SW_M: JP8.1, Q2.1, R1.1
- net +3V3: now also C22.1, U$3.4
- net +3V3_XBEE: now also Q2.3, SJ3.1; no longer C16.1, C17.1, U3.5
- net A0: now also JP11.2; no longer JP6.1
- net A1: now also JP11.3; no longer JP6.2
- net A6: now also JP4.1; no longer JP6.5
- net A7: now also JP11.1; no longer JP6.6
- net BOOST_SW: now also U5.2; no longer Q4.1, U5.26
- net D3: now also JP14.2; no longer JP5.1
- net D5: now also JP14.3; no longer JP5.3
- net D6: now also JP14.4; no longer JP5.4
- net D7: now also JP14.5; no longer JP5.5
- net D8: now also JP14.6; no longer JP5.6
- net D9: now also JP14.7, U$3.6; no longer JP5.7
- net GND: now also C22.2, JP5.2, SJ4.2, T1.2, U$3.1; no longer BAT1.GND
- net H1: now also JP14.1; no longer JP5.8
- net MISO: now also U$3.7
- net N$10: now also JP5.1; no longer BAT1.PWR@1
- net RXI: now also JP6.1
- net SCK: now also U$3.5
- net SCL: now also IC1.16, JP11.6, R10.2; no longer JP6.4
- net SDA: now also IC1.15, JP11.5, R13.2; no longer JP6.3
- net TXO: now also JP6.2
- net V+: no longer Q3.2, Q4.2, R1.1, R7.1
- net VIN: now also C18.1, C20.1, Q4.2, R16.1, U3.1, U3.3
Routing:
- net GND: track 383.9 -> 156.4 mm, vias 17 -> 39
- net +3V3: track 105.1 -> 176.2 mm, vias 5 -> 9
- net TXO: track 0.00 -> 68.2 mm, vias 0 -> 2
- net RXI: track 0.00 -> 67.6 mm, vias 0 -> 2
- net RST: track 0.00 -> 65.1 mm, vias 0 -> 2
- net A2: track 0.00 -> 51.4 mm, vias 0 -> 4
- net MOSI: track 0.00 -> 51.2 mm
- net N$6: track 48.6 -> 0.00 mm, vias 1 -> 0
- net SCK: track 0.00 -> 47.6 mm, vias 0 -> 2
- net D9: track 0.00 -> 46.7 mm, vias 0 -> 2
- net N$4: track 46.7 -> 0.00 mm, vias 1 -> 0
- net SCL: track 0.00 -> 44.7 mm, vias 0 -> 2
- net MISO: track 0.00 -> 42.1 mm, vias 0 -> 3
- net SDA: track 0.00 -> 36.6 mm
- net CS: track 0.00 -> 32.4 mm, vias 0 -> 2
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Other:
- board size 70 x 56.5 mm -> 65 x 62 mm
- board text added: "+3.7 Lipo"
- board text added: "+3V Li"
- board text added: "a0"
- board text added: "a1"
- board text added: "a3"
- board text added: "a6"
- board text added: "a7"
- board text added: "d0"
- board text added: "d1"
- board text added: "d3"
- board text added: "d5"
- board text added: "d6"
- board text added: "d7"
- board text added: "d8"
- board text added: "d9"
- board text added: "full"
- board text added: "h1"
- board text added: "on/off switch"
- board text added: "rst"
- board text added: "ss rev 03 Petre Rodan 201211"
- board text removed: "+"
- board text removed: "3.7V LiPo"
- board text removed: "CR1220"
- board text removed: "CR1225"
- board text removed: "H1"
- board text removed: "H2"
- board text removed: "L1"
- board text removed: "L2"
- board text removed: "ok"
- board text removed: "power"
- board text removed: "shtd"
- board text removed: "solar"
- board text removed: "ss rev 02 peter 201109"
- board text removed: "switch"

Commit message: latest
Parts:
- removed JP8: JUMPER-3SMD, SparkFun-Passives:SJ_3
- removed SJ3, SJ4: (no value), SparkFun-Passives:SJ_2S-TRACE
- added JP10: power, SparkFun:1X02
- added SJ345: J345, Simplex-Jumpers:SJ_4P
- added SJ6: J6, jumper:SJ
- JP4: value M01PTH -> a6
- SJ1: value (none) -> J1; device SparkFun-Passives:SJ_2S-TRACE -> jumper:SJ
- SJ2: value (none) -> J2; device SparkFun-Passives:SJ_2S-TRACE -> jumper:SJ
- moved SJ2 18.5 mm to (2.80, 32.6)
- moved C9 1.61 mm to (34.4, 16.2)
- moved U$7 1.20 mm to (31.0, 58.2)
- moved Q6 0.80 mm to (39.9, 36.0)
- moved JP3 0.41 mm to (63.1, 38.6)
- moved JP7 0.41 mm to (60.6, 38.6)
- moved Q1 0.41 mm to (56.4, 47.7)
- moved C21 0.40 mm to (11.6, 37.9)
- moved SJ1 0.40 mm to (8.20, 37.9)
- moved JP12 0.30 mm to (60.6, 56.9)
- moved JP13 0.30 mm to (63.1, 56.9)
- moved LED2 0.10 mm to (4.70, 1.60)
Connections:
- removed net A2: JP8.2, JP8.3, U5.25
- removed net N$100: C16.1, C17.1, Q2.2, R1.2, SJ3.2, U3.5
- removed net N$18: SJ2.2, U$2.6
- removed net N$20: R8.2, SJ2.1
- new net N$7: R8.2, SJ6.1, SJ6.2, U$2.6
- net +3V3_XBEE: now also C16.1, C17.1, Q2.2, R1.2, SJ2.1, SJ2.2, U3.5; no longer SJ3.1
- net GND: now also JP10.1, SJ345.4; no longer SJ4.2
- net N$12: now also JP10.2
- net XBEE_HIB: now also SJ345.2, SJ345.3, U5.25; no longer SJ4.1
- net XBEE_PWR_SW_M: now also SJ345.1; no longer JP8.1
Routing:
- net XBEE_HIB: track 2.62 -> 55.3 mm, vias 0 -> 4
- net A2: track 51.4 -> 0.00 mm, vias 4 -> 0
- net +3V3_XBEE: track 15.0 -> 32.3 mm
- net N$100: track 16.3 -> 0.00 mm
- net GND: track 156.4 -> 163.3 mm
- net N$7: track 0.00 -> 6.19 mm
- net N$12: track 39.4 -> 44.5 mm, vias 4 -> 0
- net V+: track 74.2 -> 70.7 mm
- net N$18: track 2.60 -> 0.00 mm
- net N$16: track 15.6 -> 17.9 mm
- net N$20: track 1.89 -> 0.00 mm
- net N$15: track 18.1 -> 16.6 mm
- net N$1: track 5.28 -> 6.08 mm
- net H1: track 19.0 -> 18.3 mm
- net N$13: track 2.98 -> 2.31 mm
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Other:
- board text added: "+3.7v Lipo"
- board text added: "+5v"
- board text added: "J1"
- board text added: "J2"
- board text added: "J3 4 5"
- board text added: "J6"
- board text added: "pw sw"
- board text added: "rssi"
- board text removed: "+3.7 Lipo"
- board text removed: "-"
- board text removed: "on/off switch"
- board text removed: "rst"

Commit message: latest
Parts:
- removed X1: USBSMD, SparkFun-Connectors:USB-MINIB
- moved JP10 19.8 mm to (15.2, 10.9), turned to 0 degrees
- moved LED2 18.3 mm to (22.9, 3.70), turned to 0 degrees
- moved LED1 16.6 mm to (21.3, 3.70), turned to 0 degrees
- moved R5 14.9 mm to (19.4, 3.70), turned to 90 degrees
- moved JP2 12.8 mm to (29.4, 15.6)
- moved LED4 9.43 mm to (11.7, 11.1)
- moved SJ6 8.63 mm to (4.00, 11.1), turned to 180 degrees
- moved C9 8.13 mm to (30.1, 9.30), turned to 270 degrees
- moved JP12 7.20 mm to (60.5, 49.7)
- moved JP13 7.20 mm to (63.1, 49.7)
- moved C4 6.04 mm to (52.7, 32.1)
- moved C2 6.00 mm to (49.6, 35.4)
- moved IC1 6.00 mm to (31.6, 27.2)
- moved C1 6.00 mm to (49.5, 33.4)
- moved C22 6.00 mm to (4.00, 47.6)
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Connections:
- removed net N$23: LED4.A, R8.1
- new net N$6: LED4.C, R8.2
- net GND: now also R8.1, SJ6.1, SJ6.2; no longer LED4.C, X1.GND
- net N$12: no longer X1.VBUS
- net N$7: now also LED4.A; no longer R8.2, SJ6.1, SJ6.2
Routing:
- net GND: track 163.3 -> 128.2 mm, vias 39 -> 42
- net N$12: track 44.5 -> 26.6 mm
- net N$15: track 16.6 -> 10.6 mm
- net N$16: track 17.9 -> 13.1 mm
- net N$7: track 6.19 -> 2.83 mm
- net VIN: track 99.3 -> 96.6 mm
- net BOOST_IN: track 52.2 -> 50.2 mm
- net V+: track 70.7 -> 68.8 mm, vias 2 -> 6
- net N$23: track 1.85 -> 0.00 mm
- net N$6: track 0.00 -> 1.81 mm
- net N$3: track 18.1 -> 16.3 mm
- net +3V3_XBEE: track 32.3 -> 33.7 mm
- net RST: track 64.7 -> 63.5 mm
- net XBEE_HIB: track 55.3 -> 54.1 mm
- net XBEE_PWR_SW_M: track 18.2 -> 19.3 mm
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Other:
- board size 65 x 62 mm -> 65 x 56 mm
- board text added: "+3v7"
- board text added: "ch"
- board text added: "fl"
- board text added: "power"
- board text added: "switch"
- board text removed: "+3.7v Lipo"
- board text removed: "charging"
- board text removed: "full"
- board text removed: "pw sw"

Commit message: hopefully flawless
Parts:
- removed Q2: si2305cd, Simplex-DiscreteSemi:SOT23-3_POWER
- removed R1: 100k, rcl:R0805W
- added Q3: si2305cd, Simplex-DiscreteSemi:SOT23-3_POWER
- added R17: 1M, rcl:R0805W
- added R18: 100k, rcl:R0805W
- added T2: BC846, transistor:SOT23
- R7: value 100k -> 1M
- moved SJ2 15.1 mm to (18.3, 28.9), turned to 270 degrees
- moved C20 8.30 mm to (9.70, 26.1)
- moved C18 6.67 mm to (10.1, 29.2), turned to 180 degrees
- moved C16 6.00 mm to (4.40, 27.1)
- moved C19 6.00 mm to (7.50, 26.1)
- moved U3 6.00 mm to (4.50, 23.6)
- moved C9 5.79 mm to (35.5, 11.4)
- moved C17 5.60 mm to (4.90, 29.2)
- moved R15 3.81 mm to (7.20, 4.40), turned to 270 degrees
- moved C14 2.62 mm to (26.4, 9.50)
- moved R6 2.42 mm to (33.4, 11.4)
- moved C15 1.91 mm to (18.0, 7.80)
- moved C5 1.79 mm to (11.9, 8.80), turned to 0 degrees
- moved LED2 1.60 mm to (24.5, 3.70)
- moved R5 1.60 mm to (21.0, 3.70)
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Connections:
- new net N$18: R17.1, T2.1
- new net N$20: Q3.1, R18.2, T2.3
- net +3V3_XBEE: no longer Q2.2, Q2.3, R1.2, SJ2.1, SJ2.2
- net GND: now also T2.2
- net VIN: now also Q3.2, Q3.3, R18.1, SJ2.1, SJ2.2
- net XBEE_PWR_SW_M: now also R17.2; no longer Q2.1, R1.1
Routing:
- net VIN: track 96.6 -> 114.7 mm, vias 5 -> 4
- net XBEE_PWR_SW_M: track 19.3 -> 4.45 mm
- net GND: track 128.2 -> 114.2 mm
- net +3V3_XBEE: track 33.7 -> 19.8 mm
- net N$20: track 0.00 -> 4.53 mm
- net +3V3: track 176.4 -> 173.7 mm
- net V+: track 68.8 -> 66.5 mm
- net N$18: track 0.00 -> 1.95 mm
- net N$11: track 3.83 -> 5.06 mm
- net N$9: track 3.43 -> 2.34 mm
- net +5V: track 70.4 -> 70.9 mm
- net XBEE_HIB: track 54.1 -> 54.6 mm, vias 4 -> 6
Other:
- board text added: "+3v"
- board text added: "ok"
- board text added: "power sw"
- board text added: "sck"
- board text added: "t+"
- board text added: "t-"
- board text removed: "+3V Li"
- board text removed: "fl"
- board text removed: "power"
- board text removed: "switch"
